File: KiCAD/C3Jr_v2/c3jr_v2-Aux.sch (KiCad schematic (older format))
At the start: 58 parts, among them J1 V_IN, J2 V_IN, J3 V_IN, K1 PWR SEL, K3 7Seg_Sel, K4 SCL, K5 SDA, P1 7SegDisp, P10 CONN_1, P11 CONN_1, P13 ISP, P14 CONN_1, P15 CONN_1, P24 DIL6, P25 DIL6, P26 DIL6, P27 DIL6, P28 DIL6, P29 DIL6, P30 DIL6, P31 DIL6, P32 DIL6, P33 DIL6, P34 DIL6, P35 DIL6, P36 DIL6, P37 DIL6, P38 DIL6, P39 DIL6, P41 STACK-L, P42 STACK-R, P49 CONN_1, P50 CONN_1, P51 CONN_1, P52 CONN_1, P53 CONN_1, P54 CONN_1, P7 FTDI, P8 CONN_1, P9 CONN_1, U2 7805, U6 DS3231N

Commit message: kicad cleanup
Parts:
- BT1: symbol BATT_RTC -> C3Jr_v2:Batt_RTC
- C1, C2, C8: symbol CP1 -> C3Jr_v2:CP1
- C10, C4, C7, C9: symbol C -> C3Jr_v2:C
- CD1, CD2, CD3, P41, P42: symbol CONN_4 -> C3Jr_v2:CONN_4
- D260: symbol LED -> C3Jr_v2:LED
- J1: symbol MINI-USB -> C3Jr_v2:MINI-USB
- J2: symbol USB-B -> C3Jr_v2:USB-B
- J3, K4, K5: symbol CONN_2 -> C3Jr_v2:CONN_2
- K1, K3: symbol CONN_3 -> C3Jr_v2:CONN_3
- P1: symbol CONN_8 -> C3Jr_v2:CONN_8
- P10, P11, P14, P15, P49, P50, P51, P52, P53, P54, P8, P9: symbol CONN_1 -> C3Jr_v2:CONN_1
- P13, P7: symbol CONN_6 -> C3Jr_v2:CONN_6
- P24, P25, P26, P27, P28, P29, P30, P31, P32, P33, P34, P35, P36, P37, P38, P39: symbol DIL6 -> C3Jr_v2:DIL6
- R26, R36, R37, R38: symbol R -> C3Jr_v2:R
- U2: symbol 7805 -> C3Jr_v2:7805
- U6: symbol DS3231N -> C3Jr_v2:DS3231N
Connections:
- wire segments 260 -> 363
