File: KiCAD/C3Jr_v2/c3jr_v2-LED.sch (KiCad schematic (older format))
At the start: 161 parts, among them K2 LED_ENABLE, Q1 2N5401, Q10 2N5401, Q11 2N5401, Q12 2N5401, Q13 2N5401, Q14 2N5401, Q15 2N5401, Q16 2N5401, Q2 2N5401, Q3 2N5401, Q4 2N5401, Q5 2N5401, Q6 2N5401, Q7 2N5401, Q8 2N5401, Q9 2N5401

Commit message: kicad cleanup
Parts:
- D1, D10, D100, D101, D102, D103, D104, D105, D106, D107, D108, D109, D11, D110, D111, D112, D113, D114, D115, D116, D117, D118, D119, D12, D120, D121, D122, D123, D124, D125, D126, D127, D128, D13, D14, D15, D16, D17, D18, D19, D2, D20, D21, D22, D23, D24, D25, D26, D27, D28, D29, D3, D30, D31, D32, D33, D34, D35, D36, D37, D38, D39, D4, D40, D41, D42, D43, D44, D45, D46, D47, D48, D49, D5, D50, D51, D52, D53, D54, D55, D56, D57, D58, D59, D6, D60, D61, D62, D63, D64, D65, D66, D67, D68, D69, D7, D70, D71, D72, D73, D74, D75, D76, D77, D78, D79, D8, D80, D81, D82, D83, D84, D85, D86, D87, D88, D89, D9, D90, D91, D92, D93, D94, D95, D96, D97, D98, D99: symbol LED -> C3Jr_v2:LED
- K2: symbol CONN_3 -> C3Jr_v2:CONN_3
- Q1, Q10, Q11, Q12, Q13, Q14, Q15, Q16, Q2, Q3, Q4, Q5, Q6, Q7, Q8, Q9: symbol PNP -> C3Jr_v2:PNP
- R1, R10, R11, R12, R13, R14, R15, R16, R2, R3, R4, R5, R6, R7, R8, R9: symbol R -> C3Jr_v2:R
