File: KiCAD/C3Jr_v2/c3jr_v2-mech.sch (KiCad schematic (older format))
At the start: 4 parts

Commit message: kicad cleanup
Parts:
- BF1: symbol BAFFLE -> C3Jr_v2:BAFFLE
- BP1, FP1: symbol DIFFUSER -> C3Jr_v2:DIFFUSER
- FM1: symbol FRAME -> C3Jr_v2:Frame
Changed lines of the file:
@@
-EESchema Schematic File Version 2  date 2/18/2012 10:21:07 AM
-LIBS:C3Jr_v2
-LIBS:power
+EESchema Schematic File Version 4
 LIBS:c3jr_v2-cache
-LIBS:c3jr_v2-cache
-EELAYER 25  0
+EELAYER 26 0
 EELAYER END
-$Descr A4 11700 8267
+$Descr A4 11693 8268
 encoding utf-8
 Sheet 3 4
@@
 $EndDescr
 $Comp
-L FRAME FM1
+L C3Jr_v2:Frame FM1
 U 1 1 4DC15770
 P 6350 2100
@@
 F 1 "FRAME" H 6350 2250 60  0000 C CNN
 F 2 "Frame" H 6350 2100 60  0001 C CNN
+F 3 "" H 6350 2100 50  0001 C CNN
 	1    6350 2100
 	1    0    0    -1
 $EndComp
 $Comp
-L DIFFUSER BP1
+L C3Jr_v2:DIFFUSER BP1
 U 1 1 4DC14DC7
 P 8950 3850
@@
 F 1 "BackPlate" H 8950 4000 60  0000 C CNN
 F 2 "BackPlate" H 8950 3850 60  0001 C CNN
+F 3 "" H 8950 3850 50  0001 C CNN
 	1    8950 3850
 	1    0    0    -1
 $EndComp
 $Comp
-L DIFFUSER FP1
+L C3Jr_v2:DIFFUSER FP1
 U 1 1 4DC14DC3
 P 3450 3850
@@
 F 1 "FacePlate" H 3450 4000 60  0000 C CNN
 F 2 "FacePlate" H 3450 3850 60  0001 C CNN
+F 3 "" H 3450 3850 50  0001 C CNN
 	1    3450 3850
 	1    0    0    -1
 $EndComp
 $Comp
-L BAFFLE BF1
+L C3Jr_v2:BAFFLE BF1
 U 1 1 4DC14DAD
 P 6300 3800
@@
 F 1 "BAFFLE" H 6300 4450 60  0000 C CNN
 F 2 "Baffle" H 6300 3800 60  0001 C CNN
+F 3 "" H 6300 3800 50  0001 C CNN
 	1    6300 3800
 	1    0    0    -1
