File: KiCAD/C3Jr_v2/c3jr_v2.sch (KiCad schematic (older format))
At the start: 41 parts, among them P43 CONN_1, Q17 2N5401, SW1 INC, SW12 INC, SW2 DEC, SW22 DEC, SW3 MODE, SW32 MODE, SW4 RST, SW42 RST, SW5 ENTER, SW52 ENTER, U1 STP8DP05, U3 ATMEGA8-P, U4 74HC154, X1 16MHz

Commit message: kicad cleanup
Parts:
- C11, C12, C3, C5, C6: symbol C -> C3Jr_v2:C
- D258: symbol LED -> C3Jr_v2:LED
- DIL-U1: symbol STP16DP05 -> C3Jr_v2:STP16DP05
- P43, rowBoB1: symbol CONN_1 -> C3Jr_v2:CONN_1
- PCB1: symbol PCB -> C3Jr_v2:PCB
- Q17: symbol PNP -> C3Jr_v2:PNP
- R17, R18, R19, R20, R21, R22, R23, R24, R25, R30, R31, R32, R33, R35: symbol R -> C3Jr_v2:R
- R34: symbol RVAR -> C3Jr_v2:RVAR
- SP1: symbol SPEAKER -> C3Jr_v2:SPEAKER
- SW1, SW12, SW2, SW22, SW3, SW32, SW4, SW42, SW5, SW52: symbol SW_PUSH -> C3Jr_v2:SW_PUSH
- U1: symbol STP8DP05 -> C3Jr_v2:STP8DP05
- U3: symbol ATMEGA8-P -> C3Jr_v2:ATMEGA8-P
- U4: symbol 74LS154 -> C3Jr_v2:74LS154
- X1: symbol CRYSTAL -> C3Jr_v2:CRYSTAL
